File: rgb7breakout.sch (KiCad schematic (older format))
At the start: 8 parts, among them J1 RGB7Breakout_Connector, U1 TLC5947DAP

Commit message: add fiducials to schematic
Parts:
- added FID1, FID2, FID3: FIDUCIAL_0.5MM, MF_Aesthetics:MF_Aesthetics-FIDUCIAL_0.5MM, symbol FIDUCIAL_0.5MM
Changed lines of the file:
@@
 LIBS:valves
 LIBS:myLibrary
+LIBS:MF_Aesthetics
 LIBS:rgb7breakout-cache
 EELAYER 25 0
@@
 	2450 4700 2300 4700
 Connection ~ 2300 4700
+$Comp
+L FIDUCIAL_0.5MM FID1
+U 1 1 59B974D6
+P 1600 6900
+F 0 "FID1" H 1600 6900 45  0000 R TNN
+F 1 "FIDUCIAL_0.5MM" H 1600 6840 45  0000 R TNN
+F 2 "MF_Aesthetics:MF_Aesthetics-FIDUCIAL_0.5MM" H 1630 7050 20  0001 C CNN
+F 3 "" H 1600 6900 60  0000 C CNN
+	1    1600 6900
+	1    0    0    -1
+$EndComp
+$Comp
+L FIDUCIAL_0.5MM FID2
+U 1 1 59B97508
+P 1600 7100
+F 0 "FID2" H 1600 7100 45  0000 R TNN
+F 1 "FIDUCIAL_0.5MM" H 1600 7040 45  0000 R TNN
+F 2 "MF_Aesthetics:MF_Aesthetics-FIDUCIAL_0.5MM" H 1630 7250 20  0001 C CNN
+F 3 "" H 1600 7100 60  0000 C CNN
+	1    1600 7100
+	1    0    0    -1
+$EndComp
+$Comp
+L FIDUCIAL_0.5MM FID3
+U 1 1 59B9753D
+P 1600 7300
+F 0 "FID3" H 1600 7300 45  0000 R TNN
+F 1 "FIDUCIAL_0.5MM" H 1600 7240 45  0000 R TNN
+F 2 "MF_Aesthetics:MF_Aesthetics-FIDUCIAL_0.5MM" H 1630 7450 20  0001 C CNN
+F 3 "" H 1600 7300 60  0000 C CNN
+	1    1600 7300
+	1    0    0    -1
+$EndComp
 $EndSCHEMATC

Commit message: add fiducials on back side of board, too
Parts:
- added FID4, FID5, FID6: FIDUCIAL_0.5MM, MF_Aesthetics:MF_Aesthetics-FIDUCIAL_0.5MM, symbol FIDUCIAL_0.5MM
Other:
- note added: "Board Back"
- note added: "Board Front"
Changed lines of the file:
@@
 	1    0    0    -1
 $EndComp
+$Comp
+L FIDUCIAL_0.5MM FID4
+U 1 1 59B984A1
+P 2300 6900
+F 0 "FID4" H 2300 6900 45  0000 R TNN
+F 1 "FIDUCIAL_0.5MM" H 2300 6840 45  0000 R TNN
+F 2 "MF_Aesthetics:MF_Aesthetics-FIDUCIAL_0.5MM" H 2330 7050 20  0001 C CNN
+F 3 "" H 2300 6900 60  0000 C CNN
+	1    2300 6900
+	1    0    0    -1
+$EndComp
+$Comp
+L FIDUCIAL_0.5MM FID5
+U 1 1 59B984DD
+P 2300 7100
+F 0 "FID5" H 2300 7100 45  0000 R TNN
+F 1 "FIDUCIAL_0.5MM" H 2300 7040 45  0000 R TNN
+F 2 "MF_Aesthetics:MF_Aesthetics-FIDUCIAL_0.5MM" H 2330 7250 20  0001 C CNN
+F 3 "" H 2300 7100 60  0000 C CNN
+	1    2300 7100
+	1    0    0    -1
+$EndComp
+$Comp
+L FIDUCIAL_0.5MM FID6
+U 1 1 59B98519
+P 2300 7300
+F 0 "FID6" H 2300 7300 45  0000 R TNN
+F 1 "FIDUCIAL_0.5MM" H 2300 7240 45  0000 R TNN
+F 2 "MF_Aesthetics:MF_Aesthetics-FIDUCIAL_0.5MM" H 2330 7450 20  0001 C CNN
+F 3 "" H 2300 7300 60  0000 C CNN
+	1    2300 7300
+	1    0    0    -1
+$EndComp
+Text Notes 1050 6850 0    60   ~ 0
+Board Front
+Text Notes 1750 6850 0    60   ~ 0
+Board Back
 $EndSCHEMATC

Commit message: switch back to Illinois Capacitor
Parts:
- C1: Description Capacitor Aluminum Electrolytic 6.3mm 100uF 20% 35V -> CAP ALUM 100UF 20% 16V SMD; ManufacturerPartNumber MF-CAP-6.3MM-100uF -> 107SML016M
Changed lines of the file:
@@
 F 2 "Capacitors_SMD:CP_Elec_6.3x7.7" H 6400 1900 50  0001 C CNN
 F 3 "" H 6400 1900 50  0001 C CNN
-F 4 "MF-CAP-6.3MM-100uF" H 6400 1900 60  0001 C CNN "ManufacturerPartNumber"
-F 5 "Capacitor Aluminum Electrolytic 6.3mm 100uF 20% 35V" H 6400 1900 60  0001 C CNN "Description"
+F 4 "107SML016M" H 6400 1900 60  0001 C CNN "ManufacturerPartNumber"
+F 5 "CAP ALUM 100UF 20% 16V SMD" H 6400 1900 60  0001 C CNN "Description"
 	1    6400 1900
 	1    0    0    -1

Commit message: fill out manufacturer part numbers
Parts:
- D1: Description (none) -> Single Digit 7-segment RGB LED Display, 1-inch digit height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; ManufacturerPartNumber (none) -> AD-121F2
- J1: Description (none) -> CONN HEADER .100\" SNGL R/A 8POS; ManufacturerPartNumber (none) -> PRPC008SBAN-M71RC
- U1: Description (none) -> 24-Channel, 12-Bit PWM LED Driver, HTSSOP; ManufacturerPartNumber (none) -> TLC5947DAP
Changed lines of the file:
@@
 F 2 "myLibrary:AD-121F2" H 7900 3900 50  0001 C CNN
 F 3 "" H 7900 3900 50  0001 C CNN
+F 4 "AD-121F2" H 7900 3900 60  0001 C CNN "ManufacturerPartNumber"
+F 5 "Single Digit 7-segment RGB LED Display, 1-inch digit height, common anode" H 7900 3900 60  0001 C CNN "Description"
 	1    7900 3900
 	1    0    0    -1
@@
 F 2 "myLibrary:HTSSOP-32_6.1x11mm_Pitch0.65mm_ThermalPad" H 3500 4000 50  0001 C CNN
 F 3 "" H 3500 4000 50  0001 C CNN
+F 4 "TLC5947DAP" H 3500 4000 60  0001 C CNN "ManufacturerPartNumber"
+F 5 "24-Channel, 12-Bit PWM LED Driver, HTSSOP" H 3500 4000 60  0001 C CNN "Description"
 	1    3500 4000
 	1    0    0    -1
@@
 F 2 "Pin_Headers:Pin_Header_Angled_1x08_Pitch2.54mm" H 1700 3900 60  0001 C CNN
 F 3 "" H 1700 3900 60  0001 C CNN
+F 4 "PRPC008SBAN-M71RC" H 1700 3900 60  0001 C CNN "ManufacturerPartNumber"
+F 5 "CONN HEADER .100\" SNGL R/A 8POS" H 1700 3900 60  0001 C CNN "Description"
 	1    1700 3900
 	1    0    0    -1

Commit message: rename ManufacturerPartNumber to mpn
Parts:
- C1: Description CAP ALUM 100UF 20% 16V SMD -> (none); ManufacturerPartNumber 107SML016M -> (none); description (none) -> CAP ALUM 100UF 20% 16V SMD; mpn (none) -> 107SML016M
- C2: Description Capacitor MLCC 0603 0.1uF 10% 25V -> (none); ManufacturerPartNumber MF-CAP-0603-0.1uF -> (none); description (none) -> Capacitor MLCC 0603 0.1uF 10% 25V; mpn (none) -> MF-CAP-0603-0.1uF
- D1: Description Single Digit 7-segment RGB LED Display, 1-inch digit height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 -> (none); ManufacturerPartNumber AD-121F2 -> (none); description (none) -> Single Digit 7-segment RGB LED Display, 1-inch digit height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; mpn (none) -> AD-121F2
- D2: Description LED RGB DIFFUSED 4LCC SMD -> (none); ManufacturerPartNumber CLV1A-FKB-CHMKPEHBB7A363 -> (none); description (none) -> LED RGB DIFFUSED 4LCC SMD; mpn (none) -> CLV1A-FKB-CHMKPEHBB7A363
- J1: Description CONN HEADER .100\" SNGL R/A 8POS -> (none); ManufacturerPartNumber PRPC008SBAN-M71RC -> (none); description (none) -> CONN HEADER .100\" SNGL R/A 8POS; mpn (none) -> PRPC008SBAN-M71RC
- R1: Description RES SMD 2.49K OHM 1% 1/10W 0603 -> (none); ManufacturerPartNumber RC0603FR-072K49L -> (none); description (none) -> RES SMD 2.49K OHM 1% 1/10W 0603; mpn (none) -> RC0603FR-072K49L
- R2: Description Resistor Thick Film 0603 10K Ohm 5% 100mW 75V -> (none); ManufacturerPartNumber MF-RES-0603-10K -> (none); description (none) -> Resistor Thick Film 0603 10K Ohm 5% 100mW 75V; mpn (none) -> MF-RES-0603-10K
- U1: Description 24-Channel, 12-Bit PWM LED Driver, HTSSOP -> (none); ManufacturerPartNumber TLC5947DAP -> (none); description (none) -> 24-Channel, 12-Bit PWM LED Driver, HTSSOP; mpn (none) -> TLC5947DAP
Changed lines of the file:
@@
 F 2 "myLibrary:AD-121F2" H 7900 3900 50  0001 C CNN
 F 3 "" H 7900 3900 50  0001 C CNN
-F 4 "AD-121F2" H 7900 3900 60  0001 C CNN "ManufacturerPartNumber"
-F 5 "Single Digit 7-segment RGB LED Display, 1-inch digit height, common anode" H 7900 3900 60  0001 C CNN "Description"
+F 4 "AD-121F2" H 7900 3900 60  0001 C CNN "mpn"
+F 5 "Single Digit 7-segment RGB LED Display, 1-inch digit height, common anode" H 7900 3900 60  0001 C CNN "description"
 	1    7900 3900
 	1    0    0    -1
@@
 F 2 "myLibrary:HTSSOP-32_6.1x11mm_Pitch0.65mm_ThermalPad" H 3500 4000 50  0001 C CNN
 F 3 "" H 3500 4000 50  0001 C CNN
-F 4 "TLC5947DAP" H 3500 4000 60  0001 C CNN "ManufacturerPartNumber"
-F 5 "24-Channel, 12-Bit PWM LED Driver, HTSSOP" H 3500 4000 60  0001 C CNN "Description"
+F 4 "TLC5947DAP" H 3500 4000 60  0001 C CNN "mpn"
+F 5 "24-Channel, 12-Bit PWM LED Driver, HTSSOP" H 3500 4000 60  0001 C CNN "description"
 	1    3500 4000
 	1    0    0    -1
@@
 F 2 "LEDs:LED_Cree-PLCC4" H 5100 5950 50  0001 C CNN
 F 3 "" H 5100 5950 50  0001 C CNN
-F 4 "CLV1A-FKB-CHMKPEHBB7A363" H 5100 6000 60  0001 C CNN "ManufacturerPartNumber"
-F 5 "LED RGB DIFFUSED 4LCC SMD" H 5100 6000 60  0001 C CNN "Description"
+F 4 "CLV1A-FKB-CHMKPEHBB7A363" H 5100 6000 60  0001 C CNN "mpn"
+F 5 "LED RGB DIFFUSED 4LCC SMD" H 5100 6000 60  0001 C CNN "description"
 	1    5100 6000
 	1    0    0    -1
@@
 F 2 "Pin_Headers:Pin_Header_Angled_1x08_Pitch2.54mm" H 1700 3900 60  0001 C CNN
 F 3 "" H 1700 3900 60  0001 C CNN
-F 4 "PRPC008SBAN-M71RC" H 1700 3900 60  0001 C CNN "ManufacturerPartNumber"
-F 5 "CONN HEADER .100\" SNGL R/A 8POS" H 1700 3900 60  0001 C CNN "Description"
+F 4 "PRPC008SBAN-M71RC" H 1700 3900 60  0001 C CNN "mpn"
+F 5 "CONN HEADER .100\" SNGL R/A 8POS" H 1700 3900 60  0001 C CNN "description"
 	1    1700 3900
 	1    0    0    -1
@@
 F 2 "Resistors_SMD:R_0603" V 2480 3700 50  0001 C CNN
 F 3 "" H 2550 3700 50  0001 C CNN
-F 4 "RC0603FR-072K49L" H 2550 3700 60  0001 C CNN "ManufacturerPartNumber"
-F 5 "RES SMD 2.49K OHM 1% 1/10W 0603" H 2550 3700 60  0001 C CNN "Description"
+F 4 "RC0603FR-072K49L" H 2550 3700 60  0001 C CNN "mpn"
+F 5 "RES SMD 2.49K OHM 1% 1/10W 0603" H 2550 3700 60  0001 C CNN "description"
 	1    2550 3700
 	0    1    1    0
@@
 F 2 "Capacitors_SMD:CP_Elec_6.3x7.7" H 6400 1900 50  0001 C CNN
 F 3 "" H 6400 1900 50  0001 C CNN
-F 4 "107SML016M" H 6400 1900 60  0001 C CNN "ManufacturerPartNumber"
-F 5 "CAP ALUM 100UF 20% 16V SMD" H 6400 1900 60  0001 C CNN "Description"
+F 4 "107SML016M" H 6400 1900 60  0001 C CNN "mpn"
+F 5 "CAP ALUM 100UF 20% 16V SMD" H 6400 1900 60  0001 C CNN "description"
 	1    6400 1900
 	1    0    0    -1
@@
 F 2 "Capacitors_SMD:C_0603" H 2738 5000 50  0001 C CNN
 F 3 "" H 2700 5150 50  0001 C CNN
-F 4 "MF-CAP-0603-0.1uF" H 2700 5150 60  0001 C CNN "ManufacturerPartNumber"
-F 5 "Capacitor MLCC 0603 0.1uF 10% 25V" H 2700 5150 60  0001 C CNN "Description"
+F 4 "MF-CAP-0603-0.1uF" H 2700 5150 60  0001 C CNN "mpn"
+F 5 "Capacitor MLCC 0603 0.1uF 10% 25V" H 2700 5150 60  0001 C CNN "description"
 	1    2700 5150
 	1    0    0    -1
@@
 F 2 "Resistors_SMD:R_0603" V 2380 4450 50  0001 C CNN
 F 3 "" H 2450 4450 50  0001 C CNN
-F 4 "MF-RES-0603-10K" H 2450 4450 60  0001 C CNN "ManufacturerPartNumber"
-F 5 "Resistor Thick Film 0603 10K Ohm 5% 100mW 75V" H 2450 4450 60  0001 C CNN "Description"
+F 4 "MF-RES-0603-10K" H 2450 4450 60  0001 C CNN "mpn"
+F 5 "Resistor Thick Film 0603 10K Ohm 5% 100mW 75V" H 2450 4450 60  0001 C CNN "description"
 	1    2450 4450
 	1    0    0    -1
