File: rgb7breakout.kicad_pcb (KiCad board)
At the start: 2 copper layers, 26.5 x 49.5 mm, 14 parts, among them J1 RGB7Breakout_Connector, U1 TLC5947DAP

Commit message: connected up GND manually
Routing:
- net GND: track 12.7 -> 53.4 mm, vias 1 -> 2
Changed lines of the file:
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@@
   (general
     (links 75)
-    (no_connects 7)
+    (no_connects 0)
     (area 171.72819 74.3456 207.77181 135.489763)
     (thickness 1.6)
     (drawings 4)
-    (tracks 365)
+    (tracks 381)
     (zones 0)
     (modules 14)
@@
   (segment (start 199.800001 87.199999) (end 199.349999 87.650001) (width 0.5) (layer B.Cu) (net 1))
   (segment (start 199.349999 87.650001) (end 198.5 88.5) (width 0.5) (layer B.Cu) (net 1))
+  (segment (start 189.5 88.5) (end 189.799999 88.200001) (width 0.2) (layer B.Cu) (net 2))
+  (segment (start 189.799999 88.200001) (end 189.799999 83.500001) (width 0.2) (layer B.Cu) (net 2))
+  (segment (start 189.799999 83.500001) (end 192.3 81) (width 0.2) (layer B.Cu) (net 2))
+  (segment (start 192.3 81) (end 192.3 80) (width 0.2) (layer B.Cu) (net 2))
+  (segment (start 189.35 98.95) (end 189.35 88.65) (width 0.2) (layer F.Cu) (net 2))
+  (segment (start 189.35 88.65) (end 189.5 88.5) (width 0.2) (layer F.Cu) (net 2))
+  (via (at 189.5 88.5) (size 0.6) (drill 0.4) (layers F.Cu B.Cu) (net 2))
+  (segment (start 188.25 96.5) (end 188.25 94.5) (width 0.2) (layer B.Cu) (net 2))
+  (segment (start 188.05 98.95) (end 188.05 96.7) (width 0.2) (layer B.Cu) (net 2))
+  (segment (start 188.05 96.7) (end 188.25 96.5) (width 0.2) (layer B.Cu) (net 2))
+  (segment (start 193.65 98.625) (end 192.275 98.625) (width 0.2) (layer B.Cu) (net 2))
+  (segment (start 192.275 98.625) (end 191.95 98.95) (width 0.2) (layer B.Cu) (net 2))
+  (segment (start 186.3 121.5) (end 187.150001 120.649999) (width 0.2) (layer F.Cu) (net 2))
+  (segment (start 187.150001 120.649999) (end 187.150001 108.949999) (width 0.2) (layer F.Cu) (net 2))
+  (segment (start 187.150001 108.949999) (end 187.385001 108.714999) (width 0.2) (layer F.Cu) (net 2))
+  (segment (start 187.385001 108.714999) (end 188.05 108.05) (width 0.2) (layer F.Cu) (net 2))
   (segment (start 194 118.5) (end 190.25 118.5) (width 0.2) (layer B.Cu) (net 2))
   (segment (start 186.3 121.5) (end 189.3 118.5) (width 0.2) (layer F.Cu) (net 2))
